File: rgbww32c3.sch (EAGLE design)
At the start: 19 parts, among them IC2 7805TV

Commit message: adjusted channel names
Connections:
- net CH1: now also SV1.8, U$1.D; no longer SV1.4, U$3.D
- net CH2: now also SV1.7, U$1.D1; no longer SV1.5, U$2.D1
- net CH4: now also SV1.5, U$2.D1; no longer SV1.7, U$1.D1
- net CH5: now also SV1.4, U$3.D; no longer SV1.8, U$1.D
Changed lines of the file:
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@@
 <net name="CH1" class="0">
 <segment>
-<wire x1="63.5" y1="7.62" x2="142.24" y2="7.62" width="0.1524" layer="91"/>
-<pinref part="U$3" gate="G$1" pin="D"/>
-<wire x1="142.24" y1="7.62" x2="142.24" y2="22.86" width="0.1524" layer="91"/>
-<pinref part="SV1" gate="1" pin="4"/>
-<wire x1="63.5" y1="7.62" x2="63.5" y2="-7.62" width="0.1524" layer="91"/>
+<pinref part="U$1" gate="G$1" pin="D"/>
+<wire x1="53.34" y1="15.24" x2="60.96" y2="15.24" width="0.1524" layer="91"/>
+<wire x1="60.96" y1="15.24" x2="60.96" y2="22.86" width="0.1524" layer="91"/>
+<pinref part="SV1" gate="1" pin="8"/>
+<wire x1="53.34" y1="15.24" x2="53.34" y2="-7.62" width="0.1524" layer="91"/>
 </segment>
 </net>
@@
 </net>
 <net name="CH2" class="0">
-<segment>
-<wire x1="88.9" y1="22.86" x2="88.9" y2="12.7" width="0.1524" layer="91"/>
-<wire x1="88.9" y1="12.7" x2="60.96" y2="12.7" width="0.1524" layer="91"/>
-<pinref part="U$2" gate="G$1" pin="D1"/>
-<pinref part="SV1" gate="1" pin="5"/>
-<wire x1="60.96" y1="12.7" x2="60.96" y2="-7.62" width="0.1524" layer="91"/>
-</segment>
-</net>
-<net name="CH4" class="0">
 <segment>
 <wire x1="48.26" y1="22.86" x2="48.26" y2="10.16" width="0.1524" layer="91"/>
@@
 <junction x="-2.54" y="12.7"/>
 <label x="-2.54" y="17.78" size="1.4224" layer="95" rot="R90" xref="yes"/>
-</segment>
-</net>
-<net name="CH5" class="0">
-<segment>
-<pinref part="U$1" gate="G$1" pin="D"/>
-<wire x1="53.34" y1="15.24" x2="60.96" y2="15.24" width="0.1524" layer="91"/>
-<wire x1="60.96" y1="15.24" x2="60.96" y2="22.86" width="0.1524" layer="91"/>
-<pinref part="SV1" gate="1" pin="8"/>
-<wire x1="53.34" y1="15.24" x2="53.34" y2="-7.62" width="0.1524" layer="91"/>
 </segment>
 </net>
@@
 </segment>
 </net>
+<net name="CH5" class="0">
+<segment>
+<wire x1="63.5" y1="7.62" x2="142.24" y2="7.62" width="0.1524" layer="91"/>
+<pinref part="U$3" gate="G$1" pin="D"/>
+<wire x1="142.24" y1="7.62" x2="142.24" y2="22.86" width="0.1524" layer="91"/>
+<pinref part="SV1" gate="1" pin="4"/>
+<wire x1="63.5" y1="7.62" x2="63.5" y2="-7.62" width="0.1524" layer="91"/>
+</segment>
+</net>
+<net name="CH4" class="0">
+<segment>
+<wire x1="88.9" y1="22.86" x2="88.9" y2="12.7" width="0.1524" layer="91"/>
+<wire x1="88.9" y1="12.7" x2="60.96" y2="12.7" width="0.1524" layer="91"/>
+<pinref part="U$2" gate="G$1" pin="D1"/>
+<pinref part="SV1" gate="1" pin="5"/>
+<wire x1="60.96" y1="12.7" x2="60.96" y2="-7.62" width="0.1524" layer="91"/>
+</segment>
+</net>

Commit message: initial testing version
programming the ESP32 now works using an esp_prog. It does require to pull GPIO9 low, hence the extra PRG button. The auto programming function of other ESP models (GPIO0) does not work on the C3, it seems.
Parts:
- added J_PRG: 1296-T06, con-leotronics:1296-T06
- added R7: 10k, rcl:R-EU_R0805
- PRG: value 1296-T06 -> SWITCH-MOMENTARY-2SMD-1101NE; device con-leotronics:1296-T06 -> SparkFun-Electromechanical:SWITCH-MOMENTARY-2SMD-1101NE
Connections:
- new net N$1: R7.2, U$5.GP9@1
- new net N$2: PRG.2, R7.1
- net 3V3: now also J_PRG-2.B; no longer PRG-2.B
- net EN: now also J_PRG-1.B; no longer PRG-1.B
- net GND: now also J_PRG-4.B, PRG.1; no longer PRG-4.B
- net GPIO0: now also J_PRG-6.B; no longer PRG-6.B
- net RX: now also J_PRG-5.B; no longer PRG-5.B
- net TX: now also J_PRG-3.B; no longer PRG-3.B
Changed lines of the file:
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@@
 <part name="R6" library="rcl" deviceset="R-EU_" device="R0805" value="10k"/>
 <part name="GND5" library="supply1" deviceset="GND" device=""/>
-<part name="PRG" library="con-leotronics" deviceset="1296-T06" device=""/>
+<part name="J_PRG" library="con-leotronics" deviceset="1296-T06" device=""/>
 <part name="C1" library="rcl" deviceset="C-EU" device="C1206"/>
 <part name="GND6" library="SparkFun-Aesthetics" deviceset="GND" device=""/>
 <part name="C2" library="rcl" deviceset="C-EU" device="C1206"/>
 <part name="GND12" library="SparkFun-Aesthetics" deviceset="GND" device=""/>
+<part name="R7" library="rcl" deviceset="R-EU_" device="R0805" value="10k"/>
+<part name="GND13" library="supply1" deviceset="GND" device=""/>
+<part name="PRG" library="SparkFun-Electromechanical" deviceset="SWITCH-MOMENTARY-2" device="SMD-1101NE" value=""/>
 </parts>
 <sheets>
@@
 <instance part="R6" gate="G$1" x="-58.42" y="10.16" rot="R90"/>
 <instance part="GND5" gate="1" x="83.82" y="-10.16"/>
-<instance part="PRG" gate="-1" x="22.86" y="114.3"/>
-<instance part="PRG" gate="-2" x="53.34" y="114.3"/>
-<instance part="PRG" gate="-3" x="22.86" y="111.76"/>
-<instance part="PRG" gate="-4" x="53.34" y="111.76"/>
-<instance part="PRG" gate="-5" x="22.86" y="109.22"/>
-<instance part="PRG" gate="-6" x="53.34" y="109.22"/>
+<instance part="J_PRG" gate="-1" x="22.86" y="114.3"/>
+<instance part="J_PRG" gate="-2" x="53.34" y="114.3"/>
+<instance part="J_PRG" gate="-3" x="22.86" y="111.76"/>
+<instance part="J_PRG" gate="-4" x="53.34" y="111.76"/>
+<instance part="J_PRG" gate="-5" x="22.86" y="109.22"/>
+<instance part="J_PRG" gate="-6" x="53.34" y="109.22"/>
 <instance part="C1" gate="G$1" x="-10.16" y="124.46"/>
 <instance part="GND6" gate="1" x="-10.16" y="111.76"/>
 <instance part="C2" gate="G$1" x="-45.72" y="124.46"/>
 <instance part="GND12" gate="1" x="-45.72" y="111.76"/>
+<instance part="R7" gate="G$1" x="-53.34" y="5.08" rot="R90"/>
+<instance part="GND13" gate="1" x="-53.34" y="-20.32"/>
+<instance part="PRG" gate="G$1" x="-53.34" y="-7.62" smashed="yes" rot="R90">
+<attribute name="NAME" x="-50.8" y="-2.54" size="1.778" layer="95" rot="R270"/>
+<attribute name="VALUE" x="-50.8" y="-10.16" size="1.778" layer="96" rot="R90"/>
+</instance>
 </instances>
 <busses>
@@
 </segment>
 <segment>
-<pinref part="PRG" gate="-4" pin="B"/>
+<pinref part="J_PRG" gate="-4" pin="B"/>
 <wire x1="50.8" y1="111.76" x2="45.72" y2="111.76" width="0.1524" layer="91"/>
 <label x="45.72" y="111.76" size="1.4224" layer="95" rot="R180" xref="yes"/>
@@
 <pinref part="C2" gate="G$1" pin="2"/>
 <wire x1="-45.72" y1="114.3" x2="-45.72" y2="119.38" width="0.1524" layer="91"/>
+</segment>
+<segment>
+<pinref part="GND13" gate="1" pin="GND"/>
+<pinref part="PRG" gate="G$1" pin="1"/>
+<wire x1="-53.34" y1="-17.78" x2="-53.34" y2="-12.7" width="0.1524" layer="91"/>
 </segment>
 </net>
@@
 </segment>
 <segment>
-<wire x1="-58.42" y1="-7.62" x2="-53.34" y2="-7.62" width="0.1524" layer="91"/>
 <pinref part="R6" gate="G$1" pin="1"/>
 <wire x1="-58.42" y1="5.08" x2="-58.42" y2="-7.62" width="0.1524" layer="91"/>
@@
 <wire x1="-58.42" y1="-7.62" x2="-63.5" y2="-7.62" width="0.1524" layer="91"/>
 <wire x1="-63.5" y1="-7.62" x2="-63.5" y2="-5.08" width="0.1524" layer="91"/>
-<junction x="-58.42" y="-7.62"/>
 </segment>
 <segment>
@@
 </segment>
 <segment>
-<pinref part="PRG" gate="-2" pin="B"/>
+<pinref part="J_PRG" gate="-2" pin="B"/>
 <wire x1="50.8" y1="114.3" x2="45.72" y2="114.3" width="0.1524" layer="91"/>
 <label x="45.72" y="114.3" size="1.4224" layer="95" rot="R180" xref="yes"/>
@@
 </segment>
 <segment>
-<pinref part="PRG" gate="-1" pin="B"/>
+<pinref part="J_PRG" gate="-1" pin="B"/>
 <wire x1="20.32" y1="114.3" x2="15.24" y2="114.3" width="0.1524" layer="91"/>
 <label x="15.24" y="114.3" size="1.4224" layer="95" rot="R180" xref="yes"/>
@@
 <net name="TX" class="0">
 <segment>
-<pinref part="PRG" gate="-3" pin="B"/>
+<pinref part="J_PRG" gate="-3" pin="B"/>
 <wire x1="20.32" y1="111.76" x2="15.24" y2="111.76" width="0.1524" layer="91"/>
 <label x="15.24" y="111.76" size="1.4224" layer="95" rot="R180" xref="yes"/>
@@
 <pinref part="U$5" gate="G$1" pin="TX"/>
 <wire x1="-58.42" y1="83.82" x2="-58.42" y2="88.9" width="0.1524" layer="91"/>
+<label x="-58.42" y="88.9" size="1.778" layer="95" rot="R90" xref="yes"/>
 </segment>
 </net>
 <net name="RX" class="0">
 <segment>
-<pinref part="PRG" gate="-5" pin="B"/>
+<pinref part="J_PRG" gate="-5" pin="B"/>
 <wire x1="20.32" y1="109.22" x2="15.24" y2="109.22" width="0.1524" layer="91"/>
 <label x="15.24" y="109.22" size="1.4224" layer="95" rot="R180" xref="yes"/>
@@
 <pinref part="U$5" gate="G$1" pin="RX"/>
 <wire x1="-53.34" y1="83.82" x2="-53.34" y2="88.9" width="0.1524" layer="91"/>
+<label x="-53.34" y="88.9" size="1.778" layer="95" rot="R90" xref="yes"/>
 </segment>
 </net>
 <net name="GPIO0" class="0">
 <segment>
-<pinref part="PRG" gate="-6" pin="B"/>
+<pinref part="J_PRG" gate="-6" pin="B"/>
 <wire x1="50.8" y1="109.22" x2="45.72" y2="109.22" width="0.1524" layer="91"/>
 <label x="45.72" y="109.22" size="1.4224" layer="95" rot="R180" xref="yes"/>
@@
 </segment>
 </net>
+<net name="N$1" class="0">
+<segment>
+<pinref part="U$5" gate="G$1" pin="GP9@1"/>
+<pinref part="R7" gate="G$1" pin="2"/>
+<wire x1="-53.34" y1="10.16" x2="-53.34" y2="27.94" width="0.1524" layer="91"/>
+</segment>
+</net>
+<net name="N$2" class="0">
+<segment>
+<pinref part="PRG" gate="G$1" pin="2"/>
+<pinref part="R7" gate="G$1" pin="1"/>
+<wire x1="-53.34" y1="-2.54" x2="-53.34" y2="0" width="0.1524" layer="91"/>
+</segment>
+</net>

Commit message: few routing corrections to better avoid short circuits
Connections:
- net CH1S: now also R4.1, U$1.G, U$5.GP10; no longer R3.1, U$1.G1, U$5.GP7
- net CH2S: now also R3.1, U$1.G1, U$5.GP7; no longer R4.1, U$1.G, U$5.GP10
- net CH3S: now also R2.1, U$2.G, U$5.GP6; no longer R5.1, U$2.G1, U$5.GP5
- net CH4S: now also R5.1, U$2.G1, U$5.GP5; no longer R2.1, U$2.G, U$5.GP6
Changed lines of the file:
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@@
 </segment>
 </net>
-<net name="CH2S" class="0">
+<net name="CH1S" class="0">
 <segment>
 <pinref part="R4" gate="G$1" pin="1"/>
@@
 </segment>
 </net>
-<net name="CH1S" class="0">
+<net name="CH2S" class="0">
 <segment>
 <pinref part="R3" gate="G$1" pin="1"/>
@@
 </segment>
 </net>
-<net name="CH4S" class="0">
+<net name="CH3S" class="0">
 <segment>
 <pinref part="R2" gate="G$1" pin="1"/>
@@
 </segment>
 </net>
-<net name="CH3S" class="0">
+<net name="CH4S" class="0">
 <segment>
 <pinref part="R5" gate="G$1" pin="1"/>
